Commit message: save

File: description/camera.xacro (robot description, xacro)
@@ -37,6 +37,6 @@
                 <image>
                     <format>R8G8B8</format>
-                    <width>640</width>
-                    <height>480</height>
+                    <width>1920</width>
+                    <height>1088</height>
                 </image>
                 <clip>

File: description/robot_core.xacro (robot description, xacro)
@@ -2,5 +2,11 @@
 <robot xmlns:xacro="http://www.ros.org/wiki/xacro">
     <xacro:include filename="inertial_macros.xacro"/>
-<!--    Base Link-->
+    <material name="black">
+        <color rgba="0 0 0 1"/>
+    </material>
+    <material name="grey">
+        <color rgba="0 0 0 0.8"/>
+    </material>
+    <!--    Base Link-->
     <link name="base_link">
     </link>
